File: warpstone.kicad_pcb (KiCad board)
At the start: 2 copper layers, 209.6 x 76.2 mm, 91 parts, among them SW1 SW_Push, U1 ProMicro

Commit message: overhaul
total overhaul to the design of the board
case design now available
protos en route
Parts:
- removed G***: LOGO, silk stuff:thewarpstonetext
- removed MX20-ISO1: MX-NoLED, MX_Only:MXOnly-ISO-ReversedStabilizers
- D1, D10, D11, D12, D13, D14, D15, D16, D17, D18, D19, D2, D20, D21, D22, D23, D24, D25, D26, D27, D28, D29, D3, D30, D31, D32, D33, D34, D35, D36, D37, D38, D4, D5, D6, D7, D8, D9: footprint Keebio-Parts:Diode-Hybrid-Back -> Keebio-Parts:D_SOD123
- U1: moved to B.Cu
- moved U1 204.8 mm to (250.0, 45.2)
- moved SW1 192.5 mm to (250.0, 65.5)
- moved D36 16.8 mm to (189.3, 96.4), turned to 90 degrees
- moved D33 16.8 mm to (82.2, 96.4), turned to 90 degrees
- moved D34 16.2 mm to (98.8, 96.4), turned to 90 degrees
- moved D35 14.3 mm to (172.6, 96.4), turned to 90 degrees
- moved D20 7.14 mm to (238.1, 58.3), turned to 90 degrees
- moved D11 4.29 mm to (59.5, 58.3), turned to 90 degrees
- moved D12 3.37 mm to (63.1, 58.3), turned to 90 degrees
- moved D10 3.37 mm to (215.5, 39.3), turned to 90 degrees
- moved D9 2.66 mm to (211.9, 39.3), turned to 90 degrees
- moved D1 2.38 mm to (59.5, 39.3), turned to 90 degrees
- moved D13 2.38 mm to (83.3, 58.3), turned to 90 degrees
- moved D14 2.38 mm to (102.4, 58.3), turned to 90 degrees
- moved D15 2.38 mm to (121.4, 58.3), turned to 90 degrees
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Routing:
- net c10: track 251.5 -> 62.1 mm, vias 1 -> 0
- net c9: track 258.4 -> 87.2 mm, vias 1 -> 0
- net c8: track 243.4 -> 87.5 mm, vias 1 -> 0
- net c7: track 215.0 -> 76.6 mm, vias 1 -> 0
- net c6: track 205.3 -> 80.8 mm, vias 1 -> 0
- net c5: track 201.9 -> 92.6 mm, vias 1 -> 0
- net c4: track 161.7 -> 68.0 mm, vias 1 -> 0
- net r4: track 295.6 -> 207.2 mm
- net c3: track 155.8 -> 80.6 mm, vias 1 -> 0
- net c2: track 111.2 -> 75.4 mm
- net r3: track 224.7 -> 200.0 mm, vias 1 -> 0
- net r2: track 201.7 -> 178.6 mm
- net r1: track 171.9 -> 156.0 mm
- net RST: track 14.7 -> 0.00 mm
- net Net-(D34-Pad2): track 31.8 -> 42.4 mm
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Other:
- board size 209.6 x 76.2 mm -> 228.6 x 76.2 mm
