File: warpstone - diode array.kicad_pcb (KiCad board)
At the start: 2 copper layers, 565.5 x 266.7 mm, 247 parts, among them SW1 SW_Push, U1 ProMicro

Commit message: updates
some more updates n stuff
Parts:
- removed the MX1 at (-280.4, -76.8)
- removed the MX1 at (-280.4, 101.8)
- removed the MX1 at (-280.4, 12.5)
- removed the MX10 at (-99.4, -76.8)
- removed the MX10 at (-99.4, 101.8)
- removed the MX10 at (-99.4, 12.5)
- removed the MX11 at (-278.0, -57.7)
- removed the MX11 at (-278.0, 120.8)
- removed the MX11 at (-278.0, 31.6)
- removed the MX12 at (-251.8, -57.7)
- removed the MX12 at (-251.8, 120.8)
- removed the MX12 at (-251.8, 31.6)
- removed the MX13 at (-232.8, -57.7)
- removed the MX13 at (-232.8, 120.8)
- removed the MX13 at (-232.8, 31.6)
- removed the MX14 at (-213.7, -57.7)
- removed the MX14 at (-213.7, 120.8)
- removed the MX14 at (-213.7, 31.6)
- removed the MX15 at (-194.7, -57.7)
- removed the MX15 at (-194.7, 120.8)
- removed the MX15 at (-194.7, 31.6)
- removed the MX16 at (-175.6, -57.7)
- removed the MX16 at (-175.6, 120.8)
- removed the MX16 at (-175.6, 31.6)
- removed the MX17 at (-156.6, -57.7)
- removed the MX17 at (-156.6, 120.8)
- removed the MX17 at (-156.6, 31.6)
- removed the MX18 at (-137.5, -57.7)
- removed the MX18 at (-137.5, 120.8)
- removed the MX18 at (-137.5, 31.6)
- removed the MX19 at (-118.5, -57.7)
- removed the MX19 at (-118.5, 120.8)
- removed the MX19 at (-118.5, 31.6)
- removed the MX2 at (-256.6, -76.8)
- removed the MX2 at (-256.6, 101.8)
- removed the MX2 at (-256.6, 12.5)
- removed the MX20 at (-97.0, -57.7)
- removed the MX20 at (-97.0, 120.8)
- removed the MX20 at (-97.0, 31.6)
- removed the MX20-2.25u1 at (-106.6, -57.7)
- removed the MX20-2.25u1 at (-106.6, 120.8)
- removed the MX20-2.25u1 at (-106.6, 31.6)
- removed the MX21 at (-282.8, -38.7)
- removed the MX21 at (-282.8, 139.9)
- removed the MX21 at (-282.8, 50.6)
- removed the MX21-2.25u1 at (-273.2, -38.7)
- removed the MX21-2.25u1 at (-273.2, 139.9)
- removed the MX21-2.25u1 at (-273.2, 50.6)
- removed the MX22 at (-261.3, -38.7)
- removed the MX22 at (-261.3, 139.9)
- removed the MX22 at (-261.3, 50.6)
- removed the MX23 at (-242.3, -38.7)
- removed the MX23 at (-242.3, 139.9)
- removed the MX23 at (-242.3, 50.6)
- removed the MX24 at (-223.2, -38.7)
- removed the MX24 at (-223.2, 139.9)
- removed the MX24 at (-223.2, 50.6)
- removed the MX25 at (-204.2, -38.7)
- removed the MX25 at (-204.2, 139.9)
- removed the MX25 at (-204.2, 50.6)
- removed the MX26 at (-185.1, -38.7)
- removed the MX26 at (-185.1, 139.9)
- removed the MX26 at (-185.1, 50.6)
- removed the MX27 at (-166.1, -38.7)
- removed the MX27 at (-166.1, 139.9)
- removed the MX27 at (-166.1, 50.6)
- removed the MX28 at (-147.0, -38.7)
- removed the MX28 at (-147.0, 139.9)
- removed the MX28 at (-147.0, 50.6)
- removed the MX29 at (-128.0, -38.7)
- removed the MX29 at (-128.0, 139.9)
- removed the MX29 at (-128.0, 50.6)
- removed the MX3 at (-237.5, -76.8)
- removed the MX3 at (-237.5, 101.8)
- removed the MX3 at (-237.5, 12.5)
- removed the MX30 at (-101.8, -38.7)
- removed the MX30 at (-101.8, 139.9)
- removed the MX30 at (-101.8, 50.6)
- removed the MX30-2.75u1 at (-111.3, -38.7)
- removed the MX30-2.75u1 at (-111.3, 139.9)
- removed the MX30-2.75u1 at (-111.3, 50.6)
- removed the MX31 at (-282.8, -19.6)
- removed the MX31 at (-282.8, 158.9)
- removed the MX31 at (-282.8, 69.7)
- removed the MX31-1u1 at (-285.2, -19.6)
- removed the MX31-1u1 at (-285.2, 158.9)
- removed the MX31-1u1 at (-285.2, 69.7)
- removed the MX32 at (-259.0, -19.6)
- removed the MX32 at (-259.0, 158.9)
- removed the MX32 at (-259.0, 69.7)
- removed the MX32-1u1 at (-266.1, -19.6)
- removed the MX32-1u1 at (-266.1, 158.9)
- removed the MX32-1u1 at (-266.1, 69.7)
- removed the MX33 at (-235.1, -19.6)
- removed the MX33 at (-235.1, 158.9)
- removed the MX33 at (-235.1, 69.7)
- removed the MX34 at (-206.6, -19.6)
- removed the MX34 at (-206.6, 158.9)
- removed the MX34 at (-206.6, 69.7)
- removed the MX34-3u1 at (-218.5, -19.6)
- removed the MX34-3u1 at (-218.5, 158.9)
- removed the MX34-3u1 at (-218.5, 69.7)
- removed the MX34-6u1 at (-189.9, -19.6)
- removed the MX34-6u1 at (-189.9, 158.9)
- removed the MX34-6u1 at (-189.9, 69.7)
- removed the MX34-7u1 at (-189.9, -19.6)
- removed the MX34-7u1 at (-189.9, 158.9)
- removed the MX34-7u1 at (-189.9, 69.7)
- removed the MX35 at (-173.2, -19.6)
- removed the MX35 at (-173.2, 158.9)
- removed the MX35 at (-173.2, 69.7)
- removed the MX35-3u1 at (-161.3, -19.6)
- removed the MX35-3u1 at (-161.3, 158.9)
- removed the MX35-3u1 at (-161.3, 69.7)
- removed the MX36 at (-144.7, -19.6)
- removed the MX36 at (-144.7, 158.9)
- removed the MX36 at (-144.7, 69.7)
- removed the MX37 at (-120.8, -19.6)
- removed the MX37 at (-120.8, 158.9)
- removed the MX37 at (-120.8, 69.7)
- removed the MX37-1u1 at (-113.7, -19.6)
- removed the MX37-1u1 at (-113.7, 158.9)
- removed the MX37-1u1 at (-113.7, 69.7)
- removed the MX38 at (-97.0, -19.6)
- removed the MX38 at (-97.0, 158.9)
- removed the MX38 at (-97.0, 69.7)
- removed the MX38-1u1 at (-94.7, -19.6)
- removed the MX38-1u1 at (-94.7, 158.9)
- removed the MX38-1u1 at (-94.7, 69.7)
- removed the MX4 at (-218.5, -76.8)
- removed the MX4 at (-218.5, 101.8)
- removed the MX4 at (-218.5, 12.5)
- removed the MX5 at (-199.4, -76.8)
- removed the MX5 at (-199.4, 101.8)
- removed the MX5 at (-199.4, 12.5)
- removed the MX6 at (-180.4, -76.8)
- removed the MX6 at (-180.4, 101.8)
- removed the MX6 at (-180.4, 12.5)
- removed the MX7 at (-161.3, -76.8)
- removed the MX7 at (-161.3, 101.8)
- removed the MX7 at (-161.3, 12.5)
- removed the MX8 at (-142.3, -76.8)
- removed the MX8 at (-142.3, 101.8)
- removed the MX8 at (-142.3, 12.5)
- removed the MX9 at (-123.2, -76.8)
- removed the MX9 at (-123.2, 101.8)
- removed the MX9 at (-123.2, 12.5)
- removed the U1 at (-75.6, -73.2)
- removed the U1 at (-75.6, 105.4)
- removed the U1 at (-75.6, 16.1)
Other:
- board size 565.5 x 266.7 mm -> 239.9 x 88.1 mm
- net class Default removed
